File: le_of.kicad_sch (KiCad schematic)
At the start: 6 parts, among them J1 ST_Link_Connector

Commit message: Finished ST link
Parts:
- removed R1, R2, R3, R4: R, symbol Device:R
- removed TP1: TestPoint, symbol Connector:TestPoint
- added J2: ATM13-12PA-R008, Footprints:HeaderFinal, symbol ATM13-12PA-R008:ATM13-12PA-R008
- added R7, R8, R9: 20, symbol Device:R
Connections:
- net Power_distribution/V_in: now also J2.12
- net microprocessor/SWCLK: now also R7.2; no longer J1.4 (Pin_4)
- net microprocessor/SWDIO: now also R8.2; no longer J1.2 (Pin_2)
- net at J1.10 (Pin_10): now also R9.1
- new net: J1.4 (Pin_4), R7.1
- new net: J1.2 (Pin_2), R8.1
- new net microprocessor/NRST: R9.2
- no-connect marks 0 -> 4
Other:
- sheet microprocessor ports: added NRST; removed none
- note added: "4V5-24V0"

Commit message: Started adding footprints. Finished wiring up schematic
Parts:
- R7, R8, R9: footprint (none) -> Resistor_SMD:R_0805_2012Metric
Changed lines of the file:
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@@
       (effects (font (size 1.27 1.27)) (justify left))
     )
-    (property "Footprint" "" (at 57.912 125.73 90)
+    (property "Footprint" "Resistor_SMD:R_0805_2012Metric" (at 57.912 125.73 90)
       (effects (font (size 1.27 1.27)) hide)
     )
@@
       (effects (font (size 1.27 1.27)) (justify left))
     )
-    (property "Footprint" "" (at 78.232 125.73 90)
+    (property "Footprint" "Resistor_SMD:R_0805_2012Metric" (at 78.232 125.73 90)
       (effects (font (size 1.27 1.27)) hide)
     )
@@
       (effects (font (size 1.27 1.27)) (justify left))
     )
-    (property "Footprint" "" (at 68.072 125.73 90)
+    (property "Footprint" "Resistor_SMD:R_0805_2012Metric" (at 68.072 125.73 90)
       (effects (font (size 1.27 1.27)) hide)
     )
@@
     )
     (property "Footprint" "Footprints:HeaderFinal" (at 173.99 30.48 90)
-      (effects (font (size 1.27 1.27)) (justify right))
+      (effects (font (size 1.27 1.27)) (justify right) hide)
     )
     (property "Datasheet" "https://componentsearchengine.com/Datasheets/1/ATM13-12PA-R008.pdf" (at 167.64 30.48 0)

Commit message: Added library. its in the overall kicad folder for me. Added footrpint for stuff
Parts:
- J1: footprint (none) -> Connector_PinHeader_2.54mm:PinHeader_2x05_P2.54mm_Vertical
Changed lines of the file:
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@@
       (effects (font (size 1.27 1.27)))
     )
-    (property "Footprint" "" (at 148.59 113.03 0)
+    (property "Footprint" "Connector_PinHeader_2.54mm:PinHeader_2x05_P2.54mm_Vertical" (at 148.59 113.03 0)
       (effects (font (size 1.27 1.27)) hide)
     )
