File: le_of.kicad_sch (KiCad schematic)
At the start: 5 parts, among them J1 ST_Link_Connector, J2 ATM13-12PA-R008

Commit message: added net labels
Connections:
- net NSRT: now reaches J1.10 (Pin_10), R9.1
- net SWCLK: now reaches J1.4 (Pin_4), R7.1
- net SWDIO: now reaches J1.2 (Pin_2), R8.1
Changed lines of the file:
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@@
     (effects (font (size 1.27 1.27)) (justify right bottom))
+  )
+  (label "NSRT" (at 59.69 99.06 0) (fields_autoplaced)
+    (effects (font (size 1.27 1.27)) (justify left bottom))
+    (property "Signal" "" (at 59.69 100.33 0)
+      (effects (font (size 1.27 1.27) italic) (justify left))
+    )
+  )
+  (label "SWDIO" (at 69.85 110.49 0) (fields_autoplaced)
+    (effects (font (size 1.27 1.27)) (justify left bottom))
+    (property "Signal" "" (at 69.85 111.76 0)
+      (effects (font (size 1.27 1.27) italic) (justify left))
+    )
+  )
+  (label "SWCLK" (at 82.55 115.57 0) (fields_autoplaced)
+    (effects (font (size 1.27 1.27)) (justify left bottom))
+    (property "Signal" "" (at 82.55 116.84 0)
+      (effects (font (size 1.27 1.27) italic) (justify left))
+    )
+  )
+  (netclass_flag "" (length 1) (shape dot) (at 74.93 138.43 0) (fields_autoplaced)
+    (effects (font (size 1.27 1.27)) (justify left bottom))
+    (property "Netclass" "Signal" (at 75.6285 137.43 0)
+      (effects (font (size 1.27 1.27) italic) (justify left) hide)
+    )
+  )
+  (netclass_flag "" (length 1) (shape dot) (at 83.82 134.62 0) (fields_autoplaced)
+    (effects (font (size 1.27 1.27)) (justify left bottom))
+    (property "Netclass" "Signal" (at 84.5185 133.62 0)
+      (effects (font (size 1.27 1.27) italic) (justify left) hide)
+    )
+  )
+  (netclass_flag "" (length 1) (shape dot) (at 62.23 142.24 0) (fields_autoplaced)
+    (effects (font (size 1.27 1.27)) (justify left bottom))
+    (property "Netclass" "Signal" (at 62.9285 141.24 0)
+      (effects (font (size 1.27 1.27) italic) (justify left) hide)
+    )
   )
   (symbol (lib_id "power:GND") (at 137.16 120.65 0) (unit 1)
