File: microprocessor.kicad_sch (KiCad schematic)
At the start: 7 parts, among them U2 STM32G0B1REI6N

Commit message: Finished ST link
Parts:
- added C9: 100n0, Capacitor_SMD:C_0805_2012Metric, symbol Device:C_Small
- added SW2: SW_MEC_5E, Footprints:EVPBV4C1L000, symbol Switch:SW_MEC_5E
Connections:
- net GND: now also U2.40 (VSS), C9.2, SW2.3 (K), SW2.4 (A)
- net NRST: now reaches U2.12 (PF2-_NRST)
- net NRST: now also C9.1, SW2.1, SW2.2

Commit message: Started adding footprints. Finished wiring up schematic
Parts:
- C1, C2, C3, C4, C5, C6: footprint (none) -> Capacitor_SMD:C_0805_2012Metric
- U2: footprint Footprints:G0B1_V3 -> Package_QFP:LQFP-32_7x7mm_P0.8mm
Other:
- company: (none) -> Bantha Boi
- title: (none) -> PCB Test
Changed lines of the file:
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@@
 (kicad_sch (version 20230121) (generator eeschema)
   (paper "A4")
+  (title_block
+    (title "PCB Test")
+    (rev "0.0.1")
+    (company "Bantha Boi")
+  )
   (junction (at 105.41 139.7) (diameter 0) (color 0 0 0 0)
   )
@@
       (effects (font (size 1.27 1.27)) (justify left))
     )
-    (property "Footprint" "" (at 97.4852 139.7 0)
+    (property "Footprint" "Capacitor_SMD:C_0805_2012Metric" (at 97.4852 139.7 0)
       (effects (font (size 1.27 1.27)) hide)
     )
@@
       (effects (font (size 1.27 1.27)) (justify left))
     )
-    (property "Footprint" "" (at 55.5752 104.14 0)
+    (property "Footprint" "Capacitor_SMD:C_0805_2012Metric" (at 55.5752 104.14 0)
       (effects (font (size 1.27 1.27)) hide)
     )
@@
       (effects (font (size 1.27 1.27)) (justify left))
     )
-    (property "Footprint" "" (at 68.2752 104.14 0)
+    (property "Footprint" "Capacitor_SMD:C_0805_2012Metric" (at 68.2752 104.14 0)
       (effects (font (size 1.27 1.27)) hide)
     )
@@
       (effects (font (size 1.27 1.27)) (justify left))
     )
-    (property "Footprint" "" (at 72.0852 128.27 0)
+    (property "Footprint" "Capacitor_SMD:C_0805_2012Metric" (at 72.0852 128.27 0)
       (effects (font (size 1.27 1.27)) hide)
     )
@@
       (effects (font (size 1.27 1.27)) (justify left))
     )
-    (property "Footprint" "" (at 106.3752 139.7 0)
+    (property "Footprint" "Capacitor_SMD:C_0805_2012Metric" (at 106.3752 139.7 0)
       (effects (font (size 1.27 1.27)) hide)
     )
@@
       (effects (font (size 1.524 1.524)))
     )
-    (property "Footprint" "Footprints:G0B1_V3" (at 156.21 45.974 0)
+    (property "Footprint" "Package_QFP:LQFP-32_7x7mm_P0.8mm" (at 156.21 45.974 0)
       (effects (font (size 1.524 1.524)) hide)
     )
@@
       (effects (font (size 1.27 1.27)) (justify left))
     )
-    (property "Footprint" "" (at 87.3252 128.27 0)
-      (effects (font (size 1.27 1.27)) hide)
-    )
+    (property "Footprint" "Capacitor_SMD:C_0805_2012Metric" (at 87.3252 128.27 0)
+      (effects (font (size 1.27 1.27)) hide)
+    )

Commit message: Added library. its in the overall kicad folder for me. Added footrpint for stuff
Parts:
- removed SW2: SW_MEC_5E, Footprints:EVPBV4C1L000, symbol Switch:SW_MEC_5E
- added S1: EVP-BV4C1L000, EVPBV4C1L000, symbol KiCad_Plugin:EVP-BV4C1L000
Connections:
- net GND: now also S1.B1 (NO_1), S1.B2 (NO_2)
- net NRST: now also S1.A1 (COM_1), S1.A2 (COM_2)
Changed lines of the file:
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@@
   (junction (at 105.41 130.81) (diameter 0) (color 0 0 0 0)
   )
-  (junction (at 231.14 124.46) (diameter 0) (color 0 0 0 0)
+  (junction (at 227.33 118.11) (diameter 0) (color 0 0 0 0)
   )
   (junction (at 67.31 105.41) (diameter 0) (color 0 0 0 0)
@@
   (junction (at 96.52 130.81) (diameter 0) (color 0 0 0 0)
   )
+  (junction (at 260.35 115.57) (diameter 0) (color 0 0 0 0)
+  )
   (junction (at 54.61 95.25) (diameter 0) (color 0 0 0 0)
   )
-  (junction (at 220.98 124.46) (diameter 0) (color 0 0 0 0)
-  )
   (junction (at 218.44 128.27) (diameter 0) (color 0 0 0 0)
   )
@@
     (stroke (width 0) (type default))
   )
-  (wire (pts (xy 220.98 121.92) (xy 220.98 124.46))
+  (wire (pts (xy 227.33 127) (xy 227.33 118.11))
     (stroke (width 0) (type default))
   )
@@
     (stroke (width 0) (type default))
   )
+  (wire (pts (xy 227.33 118.11) (xy 228.6 118.11))
+    (stroke (width 0) (type default))
+  )
   (wire (pts (xy 107.95 52.07) (xy 113.03 52.07))
     (stroke (width 0) (type default))
@@
     (stroke (width 0) (type default))
   )
+  (wire (pts (xy 220.98 115.57) (xy 220.98 102.87))
+    (stroke (width 0) (type default))
+  )
   (wire (pts (xy 105.41 130.81) (xy 105.41 132.08))
     (stroke (width 0) (type default))
   )
+  (wire (pts (xy 260.35 115.57) (xy 259.08 115.57))
+    (stroke (width 0) (type default))
+  )
   (wire (pts (xy 208.28 128.27) (xy 218.44 128.27))
     (stroke (width 0) (type default))
@@
     (stroke (width 0) (type default))
   )
+  (wire (pts (xy 260.35 102.87) (xy 260.35 115.57))
+    (stroke (width 0) (type default))
+  )
   (wire (pts (xy 218.44 128.27) (xy 220.98 128.27))
     (stroke (width 0) (type default))
@@
     (stroke (width 0) (type default))
   )
+  (wire (pts (xy 260.35 115.57) (xy 260.35 133.35))
+    (stroke (width 0) (type default))
+  )
   (wire (pts (xy 96.52 130.81) (xy 105.41 130.81))
     (stroke (width 0) (type default))
@@
     (stroke (width 0) (type default))
   )
+  (wire (pts (xy 259.08 118.11) (xy 259.08 127))
+    (stroke (width 0) (type default))
+  )
   (wire (pts (xy 96.52 115.57) (xy 96.52 95.25))
     (stroke (width 0) (type default))
@@
     (stroke (width 0) (type default))
   )
+  (wire (pts (xy 220.98 102.87) (xy 260.35 102.87))
+    (stroke (width 0) (type default))
+  )
   (wire (pts (xy 218.44 134.62) (xy 218.44 137.16))
     (stroke (width 0) (type default))
@@
     (stroke (width 0) (type default))
   )
-  (wire (pts (xy 231.14 121.92) (xy 231.14 124.46))
-    (stroke (width 0) (type default))
-  )
   (wire (pts (xy 67.31 95.25) (xy 67.31 96.52))
     (stroke (width 0) (type default))
   )
+  (wire (pts (xy 220.98 118.11) (xy 227.33 118.11))
+    (stroke (width 0) (type default))
+  )
   (wire (pts (xy 86.36 129.54) (xy 86.36 128.27))
     (stroke (width 0) (type default))
   )
+  (wire (pts (xy 259.08 127) (xy 227.33 127))
+    (stroke (width 0) (type default))
+  )
   (wire (pts (xy 218.44 128.27) (xy 218.44 129.54))
     (stroke (width 0) (type default))
@@
     (stroke (width 0) (type default))
   )
-  (wire (pts (xy 220.98 124.46) (xy 220.98 128.27))
-    (stroke (width 0) (type default))
-  )
   (wire (pts (xy 199.39 113.03) (xy 203.2 113.03))
     (stroke (width 0) (type default))
   )
-  (wire (pts (xy 231.14 124.46) (xy 231.14 137.16))
+  (wire (pts (xy 220.98 118.11) (xy 220.98 128.27))
+    (stroke (width 0) (type default))
+  )
+  (wire (pts (xy 228.6 115.57) (xy 220.98 115.57))
     (stroke (width 0) (type default))
   )
@@
     (effects (font (size 1.27 1.27)) (justify left))
   )
-  (symbol (lib_id "power:GND") (at 231.14 137.16 0) (unit 1)
-    (in_bom yes) (on_board yes) (dnp no) (fields_autoplaced)
-    (property "Reference" "#PWR026" (at 231.14 143.51 0)
-      (effects (font (size 1.27 1.27)) hide)
-    )
-    (property "Value" "GND" (at 231.14 142.24 0)
-      (effects (font (size 1.27 1.27)))
-    )
-    (property "Footprint" "" (at 231.14 137.16 0)
-      (effects (font (size 1.27 1.27)) hide)
-    )
-    (property "Datasheet" "" (at 231.14 137.16 0)
+  (symbol (lib_id "power:GND") (at 260.35 133.35 0) (unit 1)
+    (in_bom yes) (on_board yes) (dnp no) (fields_autoplaced)
+    (property "Reference" "#PWR026" (at 260.35 139.7 0)
+      (effects (font (size 1.27 1.27)) hide)
+    )
+    (property "Value" "GND" (at 260.35 138.43 0)
+      (effects (font (size 1.27 1.27)))
+    )
+    (property "Footprint" "" (at 260.35 133.35 0)
+      (effects (font (size 1.27 1.27)) hide)
+    )
+    (property "Datasheet" "" (at 260.35 133.35 0)
       (effects (font (size 1.27 1.27)) hide)
     )
@@
     )
   )
+  (symbol (lib_id "KiCad_Plugin:EVP-BV4C1L000") (at 228.6 115.57 0) (unit 1)
+    (in_bom yes) (on_board yes) (dnp no) (fields_autoplaced)
+    (property "Reference" "S1" (at 243.84 109.22 0)
+      (effects (font (size 1.27 1.27)))
+    )
+    (property "Value" "EVP-BV4C1L000" (at 243.84 111.76 0)
+      (effects (font (size 1.27 1.27)))
+    )
+    (property "Footprint" "EVPBV4C1L000" (at 255.27 113.03 0)
+      (effects (font (size 1.27 1.27)) (justify left) hide)
+    )
+    (property "Datasheet" "https://www.mouser.de/datasheet/2/315/Panasonic_Switch__EVP_BV_Series__030122-2933967.pdf" (at 255.27 115.57 0)
+      (effects (font (size 1.27 1.27)) (justify left) hide)
+    )
+    (property "Description" "Tactile Switches 6.5mm 6.2mm SMD Op Force 2.5N" (at 255.27 118.11 0)
+      (effects (font (size 1.27 1.27)) (justify left) hide)
+    )
+    (property "Height" "3.7" (at 255.27 120.65 0)
+      (effects (font (size 1.27 1.27)) (justify left) hide)
+    )
+    (property "Manufacturer_Name" "Panasonic" (at 255.27 123.19 0)
+      (effects (font (size 1.27 1.27)) (justify left) hide)
+    )
+    (property "Manufacturer_Part_Number" "EVP-BV4C1L000" (at 255.27 125.73 0)
+      (effects (font (size 1.27 1.27)) (justify left) hide)
+    )
+    (property "Mouser Part Number" "667-EVP-BV4C1L000" (at 255.27 128.27 0)
+      (effects (font (size 1.27 1.27)) (justify left) hide)
+    )
+    (property "Mouser Price/Stock" "https://www.mouser.co.uk/ProductDetail/Panasonic/EVP-BV4C1L000?qs=MyNHzdoqoQKwTvV8HYjCOw%3D%3D" (at 255.27 130.81 0)
+      (effects (font (size 1.27 1.27)) (justify left) hide)
+    )
+    (property "Arrow Part Number" "" (at 255.27 133.35 0)
+      (effects (font (size 1.27 1.27)) (justify left) hide)
+    )
+    (property "Arrow Price/Stock" "" (at 255.27 135.89 0)
+      (effects (font (size 1.27 1.27)) (justify left) hide)
+    )
+    (pin "A1")
+    (pin "A2")
+    (pin "B1")
+    (pin "B2")
+    (instances
+      (project "le_of"
+        (path "/b9db555f-f61b-4c4f-a974-ab644ea7d765/19333afa-631a-4c15-bd5d-1ee0b604e9e9"
+          (reference "S1") (unit 1)
+        )
+      )
+    )
+  )
   (symbol (lib_id "Device:C") (at 67.31 100.33 0) (unit 1)
     (in_bom yes) (on_board yes) (dnp no)
@@
         )
       )
-    )
-  )
-  (symbol (lib_id "Switch:SW_MEC_5E") (at 226.06 124.46 0) (unit 1)
-    (in_bom yes) (on_board yes) (dnp no) (fields_autoplaced)
-    (property "Reference" "SW2" (at 226.06 115.57 0)
-      (effects (font (size 1.27 1.27)))
-    )
-    (property "Value" "SW_MEC_5E" (at 226.06 118.11 0)
-      (effects (font (size 1.27 1.27)))
-    )
-    (property "Footprint" "Footprints:EVPBV4C1L000" (at 226.06 116.84 0)
-      (effects (font (size 1.27 1.27)) hide)
-    )
-    (property "Datasheet" "http://www.apem.com/int/index.php?controller=attachment&id_attachment=1371" (at 226.06 116.84 0)
-      (effects (font (size 1.27 1.27)) hide)
-    )
-    (pin "1")
-    (pin "2")
-    (pin "3")
-    (pin "4")
-    (instances
-      (project "FinalPCB"
-        (path "/731bd17f-dc7c-4e17-988a-d345d8d8464c/a481c43f-6782-4e3e-83b2-ec0cd887f9ab"
-          (reference "SW2") (unit 1)
-        )
-      )
-      (project "le_of"
-        (path "/b9db555f-f61b-4c4f-a974-ab644ea7d765/19333afa-631a-4c15-bd5d-1ee0b604e9e9"
-          (reference "SW1") (unit 1)
-        )
-      )

Commit message: Should have done a branch instead for this but oh well
Parts:
- removed S1: EVP-BV4C1L000, EVPBV4C1L000, symbol KiCad_Plugin:EVP-BV4C1L000
Changed lines of the file:
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@@
-    )
-  )
-  (symbol (lib_id "KiCad_Plugin:EVP-BV4C1L000") (at 228.6 115.57 0) (unit 1)
-    (in_bom yes) (on_board yes) (dnp no) (fields_autoplaced)
-    (property "Reference" "S1" (at 243.84 109.22 0)
-      (effects (font (size 1.27 1.27)))
-    )
-    (property "Value" "EVP-BV4C1L000" (at 243.84 111.76 0)
-      (effects (font (size 1.27 1.27)))
-    )
-    (property "Footprint" "EVPBV4C1L000" (at 255.27 113.03 0)
-      (effects (font (size 1.27 1.27)) (justify left) hide)
-    )
-    (property "Datasheet" "https://www.mouser.de/datasheet/2/315/Panasonic_Switch__EVP_BV_Series__030122-2933967.pdf" (at 255.27 115.57 0)
-      (effects (font (size 1.27 1.27)) (justify left) hide)
-    )
-    (property "Description" "Tactile Switches 6.5mm 6.2mm SMD Op Force 2.5N" (at 255.27 118.11 0)
-      (effects (font (size 1.27 1.27)) (justify left) hide)
-    )
-    (property "Height" "3.7" (at 255.27 120.65 0)
-      (effects (font (size 1.27 1.27)) (justify left) hide)
-    )
-    (property "Manufacturer_Name" "Panasonic" (at 255.27 123.19 0)
-      (effects (font (size 1.27 1.27)) (justify left) hide)
-    )
-    (property "Manufacturer_Part_Number" "EVP-BV4C1L000" (at 255.27 125.73 0)
-      (effects (font (size 1.27 1.27)) (justify left) hide)
-    )
-    (property "Mouser Part Number" "667-EVP-BV4C1L000" (at 255.27 128.27 0)
-      (effects (font (size 1.27 1.27)) (justify left) hide)
-    )
-    (property "Mouser Price/Stock" "https://www.mouser.co.uk/ProductDetail/Panasonic/EVP-BV4C1L000?qs=MyNHzdoqoQKwTvV8HYjCOw%3D%3D" (at 255.27 130.81 0)
-      (effects (font (size 1.27 1.27)) (justify left) hide)
-    )
-    (property "Arrow Part Number" "" (at 255.27 133.35 0)
-      (effects (font (size 1.27 1.27)) (justify left) hide)
-    )
-    (property "Arrow Price/Stock" "" (at 255.27 135.89 0)
-      (effects (font (size 1.27 1.27)) (justify left) hide)
-    )
-    (pin "A1")
-    (pin "A2")
-    (pin "B1")
-    (pin "B2")
-    (instances
-      (project "le_of"
-        (path "/b9db555f-f61b-4c4f-a974-ab644ea7d765/19333afa-631a-4c15-bd5d-1ee0b604e9e9"
-          (reference "S1") (unit 1)
-        )
-      )
     )
   )

Commit message: added a whole lot of footprints and layout
Parts:
- U2: footprint Package_QFP:LQFP-32_7x7mm_P0.8mm -> Package_QFP:LQFP-64-1EP_10x10mm_P0.5mm_EP5x5mm
Changed lines of the file:
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@@
       (effects (font (size 1.524 1.524)))
     )
-    (property "Footprint" "Package_QFP:LQFP-32_7x7mm_P0.8mm" (at 156.21 45.974 0)
+    (property "Footprint" "Package_QFP:LQFP-64-1EP_10x10mm_P0.5mm_EP5x5mm" (at 156.21 45.974 0)
       (effects (font (size 1.524 1.524)) hide)
     )

Commit message: idk man
Parts:
- removed U2: STM32G0B1REI6N, Package_QFP:LQFP-64-1EP_10x10mm_P0.5mm_EP5x5mm, symbol 2023-02-14_04-08-04:STM32G0B1REI6N
- added IC2: STM32G0B1RET6N, QFP50P1200X1200X160-64N, symbol Sama:STM32G0B1RET6N
- C1, C2: value 100n0 -> 4u7
- C3, C4: value 4u7 -> 100n0
Connections:
- net +3V3: now also IC2.41 (VDDIO2), IC2.6 (VBAT), IC2.7 (VREF+), IC2.8 (VDD/VDDA)
- net GND: now also IC2.40 (VSS), IC2.9 (VSS/VSSA)
- net NRST: now also IC2.12 (PF2-NRST)
- net SWCLK: now also IC2.46 (PA14-BOOT0)
- net SWDIO: now also IC2.45 (PA13)
Other:
- moved on the sheet: C9

Commit message: added bunch
Parts:
- IC2: footprint QFP50P1200X1200X160-64N -> Package_QFP:LQFP-64_10x10mm_P0.5mm
Changed lines of the file:
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@@
       (effects (font (size 1.27 1.27)))
     )
-    (property "Footprint" "QFP50P1200X1200X160-64N" (at 177.8 48.26 0)
+    (property "Footprint" "Package_QFP:LQFP-64_10x10mm_P0.5mm" (at 177.8 48.26 0)
       (effects (font (size 1.27 1.27)) (justify left) hide)
     )
