File: microprocessor.kicad_sch (KiCad schematic)
At the start: 8 parts, among them IC2 STM32G0B1RET6N

Commit message: added net labels
Parts:
- IC2: footprint Package_QFP:LQFP-64_10x10mm_P0.5mm -> QFP50P1200X1200X160-64N; Arrow Part Number STM32G0B1RET6N -> (none); Arrow Price/Stock https://www.arrow.com/en/products/stm32g0b1ret6n/stmicroele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 -> (none)

Commit message: small
Parts:
- IC2: footprint QFP50P1200X1200X160-64N -> Sama:QFP50P1200X1200X160-64N
Changed lines of the file:
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@@
       (effects (font (size 1.27 1.27)))
     )
-    (property "Footprint" "QFP50P1200X1200X160-64N" (at 177.8 145.72 0)
+    (property "Footprint" "Sama:QFP50P1200X1200X160-64N" (at 177.8 145.72 0)
       (effects (font (size 1.27 1.27)) (justify left top) hide)
     )
