File: Power_distribution.kicad_sch (KiCad schematic)
At the start: 7 parts, among them IC1 LTC3631EMS8E-3.3#PBF

Commit message: Finished ST link
Other:
- note added: "4V5-24V0"
Changed lines of the file:
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@@
     (effects (font (size 1.27 1.27)) (justify left bottom))
+  )
+  (text "4V5-24V0" (at 76.2 77.47 0)
+    (effects (font (size 1.27 1.27)) (justify right bottom))
   )
   (hierarchical_label "V_in" (shape input) (at 73.66 80.01 180) (fields_autoplaced)

Commit message: Started adding footprints. Finished wiring up schematic
Parts:
- C7, C8, C9: footprint (none) -> Capacitor_SMD:C_0805_2012Metric
- IC1: footprint SOP65P490X110-9N -> Package_SO:MSOP-8_3x3mm_P0.65mm
- L1: footprint (none) -> Inductor_SMD:L_0805_2012Metric
- R5, R6: footprint (none) -> Resistor_SMD:R_0805_2012Metric
Other:
- company: (none) -> Bantha Boi
- title: (none) -> PCB Test
Changed lines of the file:
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@@
 (kicad_sch (version 20230121) (generator eeschema)
   (paper "A4")
+  (title_block
+    (title "PCB Test")
+    (rev "0.0.1")
+    (company "Bantha Boi")
+  )
   (junction (at 101.6 85.09) (diameter 0) (color 0 0 0 0)
   )
@@
       (effects (font (size 1.27 1.27)) (justify left))
     )
-    (property "Footprint" "" (at 80.9752 87.63 0)
+    (property "Footprint" "Capacitor_SMD:C_0805_2012Metric" (at 80.9752 87.63 0)
       (effects (font (size 1.27 1.27)) hide)
     )
@@
       (effects (font (size 1.27 1.27)) (justify left))
     )
-    (property "Footprint" "" (at 158.242 76.2 90)
+    (property "Footprint" "Resistor_SMD:R_0805_2012Metric" (at 158.242 76.2 90)
       (effects (font (size 1.27 1.27)) hide)
     )
@@
       (effects (font (size 1.27 1.27)) (justify left))
     )
-    (property "Footprint" "" (at 102.5652 92.71 0)
+    (property "Footprint" "Capacitor_SMD:C_0805_2012Metric" (at 102.5652 92.71 0)
       (effects (font (size 1.27 1.27)) hide)
     )
@@
       (effects (font (size 1.27 1.27)) (justify left))
     )
-    (property "Footprint" "" (at 110.49 68.58 0)
+    (property "Footprint" "Inductor_SMD:L_0805_2012Metric" (at 110.49 68.58 0)
       (effects (font (size 1.27 1.27)) hide)
     )
@@
       (effects (font (size 1.27 1.27)) (justify left))
     )
-    (property "Footprint" "" (at 158.242 87.63 90)
+    (property "Footprint" "Resistor_SMD:R_0805_2012Metric" (at 158.242 87.63 90)
       (effects (font (size 1.27 1.27)) hide)
     )
@@
       (effects (font (size 1.27 1.27)) (justify left))
     )
-    (property "Footprint" "" (at 176.2252 76.2 0)
+    (property "Footprint" "Capacitor_SMD:C_0805_2012Metric" (at 176.2252 76.2 0)
       (effects (font (size 1.27 1.27)) hide)
     )
@@
       (effects (font (size 1.27 1.27)))
     )
-    (property "Footprint" "SOP65P490X110-9N" (at 142.24 172.39 0)
+    (property "Footprint" "Package_SO:MSOP-8_3x3mm_P0.65mm" (at 142.24 172.39 0)
       (effects (font (size 1.27 1.27)) (justify left top) hide)
     )
