File: le_of.kicad_pcb (KiCad board)
At the start: 2 copper layers, 20 parts, among them IC1 LTC3631EMS8E-3.3#PBF, J1 ST_Link_Connector, J2 ATM13-12PA-R008, U2 STM32G0B1REI6N

Commit message: idk man
Parts:
- U2: footprint Package_QFP:LQFP-32_7x7mm_P0.8mm -> Package_QFP:LQFP-64-1EP_10x10mm_P0.5mm_EP5x5mm
- moved U2 2.77 mm to (148.7, 64.1)

Commit message: added bunch
Parts:
- removed U2: STM32G0B1REI6N, Package_QFP:LQFP-64-1EP_10x10mm_P0.5mm_EP5x5mm
- added IC2: STM32G0B1RET6N, Package_QFP:LQFP-64_10x10mm_P0.5mm, F.Cu at (149.3, 64.7)
- C1, C2: value 100n0 -> 4u7
- C3, C4: value 4u7 -> 100n0
- moved C8 41.6 mm to (121.9, 85.2)
- moved C5 30.3 mm to (122.9, 71.1)
- moved R7 29.0 mm to (110.8, 63.5)
- moved J1 24.6 mm to (96.5, 58.4)
- moved IC1 22.2 mm to (128.8, 82.9)
- moved C10 21.0 mm to (122.9, 77.1)
- moved C7 19.4 mm to (119.4, 82.2)
- moved C9 19.0 mm to (122.9, 88.2)
- moved C6 18.7 mm to (122.9, 74.1), turned to 0 degrees
- moved C2 18.4 mm to (120.3, 53.3)
- moved R6 18.0 mm to (127.3, 89.6)
- moved R8 17.4 mm to (113.7, 76.8)
- moved R9 15.0 mm to (113.7, 79.8)
- moved L1 13.5 mm to (131.8, 86.6), turned to 0 degrees
- moved C3 13.5 mm to (122.9, 65.1)
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Routing:
- net /microprocessor/SWDIO: track 0.00 -> 106.1 mm
- net +3V3: track 0.00 -> 100.4 mm
- net GND: track 38.2 -> 88.9 mm

Commit message: added net labels
Parts:
- removed J2: ATM13-12PA-R008, ATM13:ATM13-12PA-R008
Routing:
- net (no net): track 0.00 -> 4.41 mm, vias 0 -> 3
Other:
- copper layers 2 -> 4

Commit message: last min save
Routing:
- net GND: track 88.9 -> 85.3 mm
- net (no net): vias 3 -> 6
Changed lines of the file:
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@@
     )
   )
+  (via (at 129.54 63.5) (size 0.8) (drill 0.4) (layers "F.Cu" "B.Cu") (net 0))
   (via (at 126.6 65.2) (size 0.8) (drill 0.4) (layers "F.Cu" "B.Cu") (net 0))
   (via (at 129.54 63.5) (size 0.8) (drill 0.4) (layers "F.Cu" "B.Cu") (net 0))
+  (via (at 129.54 63.5) (size 0.8) (drill 0.4) (layers "F.Cu" "B.Cu") (net 0))
   (via (at 126.6 65.2) (size 0.8) (drill 0.4) (layers "F.Cu" "B.Cu") (net 0))
+  (via (at 129.54 63.5) (size 0.8) (drill 0.4) (layers "F.Cu" "B.Cu") (net 0))
   (segment (start 126.6 63.9) (end 126.6 65.2) (width 0.25) (layer "In1.Cu") (net 0))
+  (segment (start 129.54 63.5) (end 127 63.5) (width 0.25) (layer "In1.Cu") (net 0))
   (segment (start 127 63.5) (end 126.6 63.9) (width 0.25) (layer "In1.Cu") (net 0))
-  (segment (start 129.54 63.5) (end 127 63.5) (width 0.25) (layer "In1.Cu") (net 0))
   (segment (start 121.92 65.1) (end 119.38 62.56) (width 0.25) (layer "F.Cu") (net 1))
   (segment (start 127 48.26) (end 121.92 48.26) (width 0.25) (layer "F.Cu") (net 1))
@@
   (segment (start 142.2 63.46) (end 143.59 63.46) (width 0.25) (layer "F.Cu") (net 1))
   (segment (start 154.94 64.96) (end 143.59 64.96) (width 0.25) (layer "F.Cu") (net 2))
-  (segment (start 113.725 81.513173) (end 113.725 76.111827) (width 0.25) (layer "F.Cu") (net 2))
-  (segment (start 122.408173 89.22) (end 121.431827 89.22) (width 0.25) (layer "F.Cu") (net 2))
-  (segment (start 113.725 76.111827) (end 99.827741 62.214568) (width 0.25) (layer "F.Cu") (net 2))
-  (segment (start 97.774568 62.214568) (end 96.52 60.96) (width 0.25) (layer "F.Cu") (net 2))
-  (segment (start 99.827741 62.214568) (end 97.774568 62.214568) (width 0.25) (layer "F.Cu") (net 2))
-  (segment (start 121.431827 89.22) (end 113.725 81.513173) (width 0.25) (layer "F.Cu") (net 2))
-  (segment (start 122.97 88.658173) (end 122.408173 89.22) (width 0.25) (layer "F.Cu") (net 2))
-  (segment (start 122.97 55.03) (end 122.97 88.658173) (width 0.25) (layer "F.Cu") (net 2))
-  (segment (start 121.28 53.34) (end 122.97 55.03) (width 0.25) (layer "F.Cu") (net 2))
+  (segment (start 121.92 89.708173) (end 121.92 91.44) (width 0.25) (layer "F.Cu") (net 2))
+  (segment (start 133.67 56.83) (end 129.54 60.96) (width 0.25) (layer "F.Cu") (net 2))
+  (segment (start 121.92 91.44) (end 91.44 91.44) (width 0.25) (layer "F.Cu") (net 2))
+  (segment (start 129.54 60.96) (end 129.54 62.775) (width 0.25) (layer "F.Cu") (net 2))
+  (segment (start 91.44 66.04) (end 96.52 60.96) (width 0.25) (layer "F.Cu") (net 2))
+  (segment (start 122.97 88.658173) (end 121.92 89.708173) (width 0.25) (layer "F.Cu") (net 2))
+  (segment (start 91.44 91.44) (end 91.44 66.04) (width 0.25) (layer "F.Cu") (net 2))
   (segment (start 131.780685 47.81) (end 146.430685 62.46) (width 0.25) (layer "F.Cu") (net 17))
   (segment (start 95.345 59.595) (end 95.345 57.245) (width 0.25) (layer "F.Cu") (net 17))

Commit message: made small changes
Parts:
- added J2: ATM13-12PA-R008, ATM13:ATM13-12PA-R008, F.Cu at (122.5, 111.1)
- IC2: footprint Package_QFP:LQFP-64_10x10mm_P0.5mm -> Sama:QFP50P1200X1200X160-64N
Connections:
- net Net-(J1-Pin_10) renamed /NSRT
- net Net-(J1-Pin_2) renamed /SWDIO
- net Net-(J1-Pin_4) renamed /SWCLK
